File: CAD/V1.0.0/Maker_Display_RGB.kicad_sch (KiCad schematic)
At the start: 58 parts, among them K1 U262-161N-4BVC11, K2 easyC-SMD, K3 JST-2pin-SMD, Q1 PMOS-SOT-23-3, SW1 YTSA007A0151803B, U1 ESP32-WROVER, U2 TPS7A2633DRVR, U3 TP4056M

Commit message: Updating open source files.
Parts:
- removed PAD? (x2): PAD_2x1.5, e-radionica.com footprinti:PAD_2x1.5, symbol e-radionica.com schematics:PAD_2x1.5
- added C? (x2): 0.1uF, e-radionica.com footprinti:0603C, symbol e-radionica.com schematics:0603C
- added D?: white, e-radionica.com footprinti:0402LED, symbol e-radionica.com schematics:0402LED
- added D?: blue, e-radionica.com footprinti:0402LED, symbol e-radionica.com schematics:0402LED
- added Q? (x2): NPN-SOT-23-3, e-radionica.com footprinti:SOT-23-3, symbol e-radionica.com schematics:NPN-SOT-23-3
- added R? (x2): 2k2, e-radionica.com footprinti:0402R, symbol e-radionica.com schematics:0402R
- added R? (x2): 10k, e-radionica.com footprinti:0603R, symbol e-radionica.com schematics:0603R
- added R? (x2): 1k, e-radionica.com footprinti:0603R, symbol e-radionica.com schematics:0603R
- added U?: CH340C, e-radionica.com footprinti:SOP-16, symbol e-radionica.com schematics:CH340C
Connections:
- net D+: now also U?.5 (UD+)
- net D-: now also U?.6 (UD-)
- net GND: now also C?.1, C?.2, U?.1 (GND)
- net IO0: now also Q?.3 (C)
- net RESET: now also Q?.3 (C)
- net RXD0: now also D?.2 (K), R?.2
- net TXD0: now also D?.2 (K), R?.2
- net VUSB: now also C?.2, R?.2, R?.2, U?.16 (VCC)
- new net: D?.1 (A), R?.1 (x2)
- new net: Q?.1 (B), R?.2 (x2)
- new net: C?.1, U?.4 (V3)
- new net: R?.1, U?.3 (RXD)
- new net: R?.1, U?.2 (TXD)
- new net DTR: Q?.2 (E), R?.1, U?.13 (DTR#)
- new net RTS: Q?.2 (E), R?.1, U?.14 (RTS#)
Other:
- note added: "Auto-reset circuit"
- note added: "CH340C USB UART"
- moved on the sheet: D1, PAD?, Q1, R3
